Commit message: Mathametically works

File: src/lawn_mower_bot/urdf/mower.urdf.xacro (robot description, xacro)
@@ -7,4 +7,9 @@
     <xacro:property name="wheel_separation" value="0.2"/>
     <xacro:property name="wheel_width" value="0.04"/>
+    <link name="dummy_link"/>
+    <joint name="dummy_joint" type="fixed">
+        <parent link="dummy_link"/>
+        <child link="base_link"/>
+    </joint>
     <!-- Base Link -->
     <link name="base_link">
@@ -31,5 +36,5 @@
         <parent link="base_link"/>
         <child link="base_footprint"/>
-        <origin xyz="0 0 0" rpy="0 0 0"/>
+        <origin xyz="0 0 -${wheel_radius}" rpy="0 0 0"/>
     </joint>
     <!-- IMU Sensor Link (attached to base_link) -->
@@ -91,8 +96,11 @@
             <wheel_separation>${wheel_separation}</wheel_separation>
             <wheel_radius>${wheel_radius}</wheel_radius>
-            <topic>cmd_vel</topic>
-            <odom_topic>odom</odom_topic>
+            <topic>/cmd_vel</topic>
+            <odom_topic>/odom</odom_topic>
             <frame_id>odom</frame_id>
             <child_frame_id>base_footprint</child_frame_id>
+            <publish_odom>true</publish_odom>
+            <publish_odom_tf>false</publish_odom_tf>
+            <publish_wheel_tf>true</publish_wheel_tf>
         </plugin>
         <!-- IMU Sensor -->

Commit message: wont move

File: src/lawn_mower_bot/urdf/mower.urdf.xacro (robot description, xacro)
@@ -1,6 +1,5 @@
 <?xml version="1.0"?>
 <robot xmlns:xacro="http://www.ros.org/wiki/xacro" name="lawn_mower_bot">
-    <!-- Constants -->
-    <xacro:property name="chassis_mass" value="10.0"/>
+    <xacro:property name="chassis_mass" value="2.0"/>
     <xacro:property name="wheel_mass" value="0.5"/>
     <xacro:property name="wheel_radius" value="0.07"/>
@@ -12,5 +11,4 @@
         <child link="base_link"/>
     </joint>
-    <!-- Base Link -->
     <link name="base_link">
         <visual>
@@ -38,5 +36,4 @@
         <origin xyz="0 0 -${wheel_radius}" rpy="0 0 0"/>
     </joint>
-    <!-- IMU Sensor Link (attached to base_link) -->
     <link name="imu_link">
       <inertial>
@@ -49,5 +46,4 @@
       <child link="imu_link"/>
     </joint>
-    <!-- Wheels -->
     <xacro:macro name="wheel_link" params="prefix">
         <link name="${prefix}_wheel">
@@ -75,5 +71,4 @@
     <xacro:wheel_link prefix="left"/>
     <xacro:wheel_link prefix="right"/>
-    <!-- Joints -->
     <joint name="left_wheel_joint" type="continuous">
         <parent link="base_link"/>
@@ -88,7 +83,33 @@
         <axis xyz="0 1 0"/>
     </joint>
-    <!-- MODERN GAZEBO PLUGINS -->
+    <link name="caster_wheel">
+        <visual>
+            <geometry>
+                <sphere radius="0.03"/>
+            </geometry>
+            <material name="white">
+                <color rgba="1.0 1.0 1.0 1.0"/>
+            </material>
+        </visual>
+        <collision>
+            <geometry>
+                <sphere radius="0.03"/>
+            </geometry>
+        </collision>
+        <inertial>
+            <mass value="0.1"/>
+            <inertia ixx="0.0001" ixy="0" ixz="0" iyy="0.0001" iyz="0" izz="0.0001"/>
+        </inertial>
+    </link>
+    <joint name="caster_joint" type="fixed">
+        <parent link="base_link"/>
+        <child link="caster_wheel"/>
+        <origin xyz="0.15 0 -0.04" rpy="0 0 0"/>
+    </joint>
+    <gazebo reference="caster_wheel">
+        <mu1>0.001</mu1>
+        <mu2>0.001</mu2>
+    </gazebo>
     <gazebo>
-        <!-- Differential Drive -->
         <plugin name="gz::sim::systems::DiffDrive" filename="gz-sim-diff-drive-system">
             <left_joint>left_wheel_joint</left_joint>
@@ -104,15 +125,12 @@
             <publish_wheel_tf>true</publish_wheel_tf>
         </plugin>
-        <!-- IMU Sensor -->
         <plugin name="gz::sim::systems::Imu" filename="gz-sim-imu-system">
             <topic>/imu/data</topic>
             <frame_id>imu_link</frame_id>
         </plugin>
-        <!-- GPS Sensor -->
         <plugin name="gz::sim::systems::NavSat" filename="gz-sim-navsat-system">
             <topic>/gps/fix</topic>
             <frame_id>base_link</frame_id>
         </plugin>
-        <!-- Publish Robot TF -->
         <plugin name="gz::sim::systems::JointStatePublisher" filename="gz-sim-joint-state-publisher-system">
             <topic>/joint_states</topic>

Commit message: Wiggle

File: src/lawn_mower_bot/urdf/mower.urdf.xacro (robot description, xacro)
@@ -4,5 +4,5 @@
     <xacro:property name="wheel_mass" value="0.5"/>
     <xacro:property name="wheel_radius" value="0.07"/>
-    <xacro:property name="wheel_separation" value="0.2"/>
+    <xacro:property name="wheel_separation" value="0.36"/>
     <xacro:property name="wheel_width" value="0.04"/>
     <link name="dummy_link"/>
@@ -13,12 +13,14 @@
     <link name="base_link">
         <visual>
+            <origin xyz="0 0 0.05" rpy="0 0 0"/>
             <geometry>
                 <box size="0.4 0.3 0.1"/>
             </geometry>
-            <material name="blue">
-                <color rgba="0.0 0.0 0.8 1.0"/>
+            <material name="red">
+                <color rgba="0.8 0.0 0.0 1.0"/>
             </material>
         </visual>
         <collision>
+            <origin xyz="0 0 0.05" rpy="0 0 0"/>
             <geometry>
                 <box size="0.4 0.3 0.1"/>
@@ -26,4 +28,5 @@
         </collision>
         <inertial>
+            <origin xyz="0 0 0.05" rpy="0 0 0"/>
             <mass value="${chassis_mass}"/>
             <inertia ixx="0.1" ixy="0.0" ixz="0.0" iyy="0.1" iyz="0.0" izz="0.1"/>
@@ -46,4 +49,32 @@
       <child link="imu_link"/>
     </joint>
+    <link name="caster_front_wheel">
+        <visual>
+            <geometry>
+                <sphere radius="0.03"/>
+            </geometry>
+            <material name="white">
+                <color rgba="1.0 1.0 1.0 1.0"/>
+            </material>
+        </visual>
+        <collision>
+            <geometry>
+                <sphere radius="0.03"/>
+            </geometry>
+        </collision>
+        <inertial>
+            <mass value="0.1"/>
+            <inertia ixx="0.0001" ixy="0" ixz="0" iyy="0.0001" iyz="0" izz="0.0001"/>
+        </inertial>
+    </link>
+    <joint name="caster_front_joint" type="fixed">
+        <parent link="base_link"/>
+        <child link="caster_front_wheel"/>
+        <origin xyz="0.15 0 -0.04" rpy="0 0 0"/>
+    </joint>
+    <gazebo reference="caster_front_wheel">
+        <mu1>0.001</mu1>
+        <mu2>0.001</mu2>
+    </gazebo>
     <xacro:macro name="wheel_link" params="prefix">
         <link name="${prefix}_wheel">
@@ -74,41 +105,15 @@
         <parent link="base_link"/>
         <child link="left_wheel"/>
-        <origin xyz="0 ${wheel_separation/2} 0" rpy="0 0 0"/>
+        <origin xyz="-0.1 ${wheel_separation/2} 0" rpy="0 0 0"/>
         <axis xyz="0 1 0"/>
+        <limit effort="20.0" velocity="10.0"/>
     </joint>
     <joint name="right_wheel_joint" type="continuous">
         <parent link="base_link"/>
         <child link="right_wheel"/>
-        <origin xyz="0 -${wheel_separation/2} 0" rpy="0 0 0"/>
+        <origin xyz="-0.1 -${wheel_separation/2} 0" rpy="0 0 0"/>
         <axis xyz="0 1 0"/>
+        <limit effort="20.0" velocity="10.0"/>
     </joint>
-    <link name="caster_wheel">
-        <visual>
-            <geometry>
-                <sphere radius="0.03"/>
-            </geometry>
-            <material name="white">
-                <color rgba="1.0 1.0 1.0 1.0"/>
-            </material>
-        </visual>
-        <collision>
-            <geometry>
-                <sphere radius="0.03"/>
-            </geometry>
-        </collision>
-        <inertial>
-            <mass value="0.1"/>
-            <inertia ixx="0.0001" ixy="0" ixz="0" iyy="0.0001" iyz="0" izz="0.0001"/>
-        </inertial>
-    </link>
-    <joint name="caster_joint" type="fixed">
-        <parent link="base_link"/>
-        <child link="caster_wheel"/>
-        <origin xyz="0.15 0 -0.04" rpy="0 0 0"/>
-    </joint>
-    <gazebo reference="caster_wheel">
-        <mu1>0.001</mu1>
-        <mu2>0.001</mu2>
-    </gazebo>
     <gazebo>
         <plugin name="gz::sim::systems::DiffDrive" filename="gz-sim-diff-drive-system">

Commit message: works with keyboard

File: src/lawn_mower_bot/urdf/mower.urdf.xacro (robot description, xacro)
@@ -1,14 +1,8 @@
 <?xml version="1.0"?>
 <robot xmlns:xacro="http://www.ros.org/wiki/xacro" name="lawn_mower_bot">
-    <xacro:property name="chassis_mass" value="2.0"/>
-    <xacro:property name="wheel_mass" value="0.5"/>
+    <xacro:property name="chassis_mass" value="2.0"/> <xacro:property name="wheel_mass" value="0.5"/>
     <xacro:property name="wheel_radius" value="0.07"/>
     <xacro:property name="wheel_separation" value="0.36"/>
     <xacro:property name="wheel_width" value="0.04"/>
-    <link name="dummy_link"/>
-    <joint name="dummy_joint" type="fixed">
-        <parent link="dummy_link"/>
-        <child link="base_link"/>
-    </joint>
     <link name="base_link">
         <visual>
@@ -17,6 +11,6 @@
                 <box size="0.4 0.3 0.1"/>
             </geometry>
-            <material name="red">
-                <color rgba="0.8 0.0 0.0 1.0"/>
+            <material name="green">
+                <color rgba="0.0 0.8 0.0 1.0"/>
             </material>
         </visual>
@@ -30,12 +24,17 @@
             <origin xyz="0 0 0.05" rpy="0 0 0"/>
             <mass value="${chassis_mass}"/>
-            <inertia ixx="0.1" ixy="0.0" ixz="0.0" iyy="0.1" iyz="0.0" izz="0.1"/>
+            <inertia ixx="0.083" ixy="0.0" ixz="0.0" iyy="0.142" iyz="0.0" izz="0.208"/>
         </inertial>
     </link>
-    <link name="base_footprint"/>
+    <link name="base_footprint">
+        <inertial>
+            <mass value="0.0001"/>
+            <inertia ixx="0.0001" ixy="0" ixz="0" iyy="0.0001" iyz="0" izz="0.0001"/>
+        </inertial>
+    </link>
     <joint name="base_footprint_joint" type="fixed">
-        <parent link="base_link"/>
-        <child link="base_footprint"/>
-        <origin xyz="0 0 -${wheel_radius}" rpy="0 0 0"/>
+        <parent link="base_footprint"/>
+        <child link="base_link"/>
+        <origin xyz="0 0 ${wheel_radius}" rpy="0 0 0"/>
     </joint>
     <link name="imu_link">
@@ -74,6 +73,7 @@
     </joint>
     <gazebo reference="caster_front_wheel">
-        <mu1>0.001</mu1>
-        <mu2>0.001</mu2>
+        <mu1>0.0</mu1>
+        <mu2>0.0</mu2>
+        <material>Gazebo/White</material>
     </gazebo>
     <xacro:macro name="wheel_link" params="prefix">
@@ -96,5 +96,5 @@
             <inertial>
                 <mass value="${wheel_mass}"/>
-                <inertia ixx="0.01" ixy="0.0" ixz="0.0" iyy="0.01" iyz="0.0" izz="0.01"/>
+                <inertia ixx="0.001" ixy="0.0" ixz="0.0" iyy="0.001" iyz="0.0" izz="0.001"/>
             </inertial>
         </link>
@@ -107,5 +107,5 @@
         <origin xyz="-0.1 ${wheel_separation/2} 0" rpy="0 0 0"/>
         <axis xyz="0 1 0"/>
-        <limit effort="20.0" velocity="10.0"/>
+        <limit effort="50.0" velocity="10.0"/>
     </joint>
     <joint name="right_wheel_joint" type="continuous">
@@ -114,6 +114,14 @@
         <origin xyz="-0.1 -${wheel_separation/2} 0" rpy="0 0 0"/>
         <axis xyz="0 1 0"/>
-        <limit effort="20.0" velocity="10.0"/>
+        <limit effort="50.0" velocity="10.0"/>
     </joint>
+    <gazebo reference="left_wheel">
+        <mu1>1.0</mu1>
+        <mu2>1.0</mu2>
+    </gazebo>
+    <gazebo reference="right_wheel">
+        <mu1>1.0</mu1>
+        <mu2>1.0</mu2>
+    </gazebo>
     <gazebo>
         <plugin name="gz::sim::systems::DiffDrive" filename="gz-sim-diff-drive-system">

Commit message: It can scan suroundings to get the map, and work in that map while trying to avoid obstracle

File: src/lawn_mower_bot/urdf/mower.urdf.xacro (robot description, xacro)
@@ -124,5 +124,107 @@
         <mu2>1.0</mu2>
     </gazebo>
+    <link name="camera_link">
+        <visual>
+            <geometry>
+                <box size="0.05 0.1 0.05"/>
+            </geometry>
+            <material name="black">
+                <color rgba="0.1 0.1 0.1 1.0"/>
+            </material>
+        </visual>
+        <collision>
+            <geometry>
+                <box size="0.05 0.1 0.05"/>
+            </geometry>
+        </collision>
+        <inertial>
+            <mass value="0.1"/>
+            <inertia ixx="0.0001" ixy="0" ixz="0" iyy="0.0001" iyz="0" izz="0.0001"/>
+        </inertial>
+    </link>
+    <!-- Mount camera at front and top of chassis block -->
+    <joint name="camera_joint" type="fixed">
+        <parent link="base_link"/>
+        <child link="camera_link"/>
+        <origin xyz="0.18 0 0.12" rpy="0 0.1 0"/> <!-- pitched slightly down -->
+    </joint>
+    <gazebo reference="camera_link">
+        <sensor type="camera" name="front_camera">
+            <update_rate>30.0</update_rate>
+            <always_on>true</always_on>
+            <visualize>true</visualize>
+            <topic>/camera/image_raw</topic>
+            <camera>
+                <horizontal_fov>1.047198</horizontal_fov> <!-- 60 degrees -->
+                <image>
+                    <width>640</width>
+                    <height>480</height>
+                    <format>R8G8B8</format>
+                </image>
+                <clip>
+                    <near>0.1</near>
+                    <far>20.0</far>
+                </clip>
+            </camera>
+        </sensor>
+    </gazebo>
+    <!-- LIDAR SENSOR -->
+    <link name="lidar_link">
+        <visual>
+            <geometry>
+                <cylinder radius="0.04" length="0.05"/>
+            </geometry>
+            <material name="blue">
+                <color rgba="0.0 0.0 0.8 1.0"/>
+            </material>
+        </visual>
+        <collision>
+            <geometry>
+                <cylinder radius="0.04" length="0.05"/>
+            </geometry>
+        </collision>
+        <inertial>
+            <mass value="0.2"/>
+            <inertia ixx="0.0001" ixy="0" ixz="0" iyy="0.0001" iyz="0" izz="0.0001"/>
+        </inertial>
+    </link>
+    <joint name="lidar_joint" type="fixed">
+        <parent link="base_link"/>
+        <child link="lidar_link"/>
+        <origin xyz="0 0 0.20" rpy="0 0 0"/>
+    </joint>
+    <gazebo reference="lidar_link">
+        <sensor name='gpu_lidar' type='gpu_lidar'>
+            <gz_frame_id>lidar_link</gz_frame_id>
+            <topic>scan</topic>
+            <update_rate>10</update_rate>
+            <ray>
+                <scan>
+                    <horizontal>
+                        <samples>640</samples>
+                        <resolution>1</resolution>
+                        <min_angle>-3.14159</min_angle>
+                        <max_angle>3.14159</max_angle>
+                    </horizontal>
+                </scan>
+                <range>
+                    <min>0.15</min>
+                    <max>12.0</max>
+                    <resolution>0.01</resolution>
+                </range>
+                <noise>
+                    <type>gaussian</type>
+                    <mean>0.0</mean>
+                    <stddev>0.01</stddev>
+                </noise>
+            </ray>
+            <always_on>1</always_on>
+            <visualize>false</visualize>
+        </sensor>
+    </gazebo>
     <gazebo>
+        <plugin name="gz::sim::systems::Sensors" filename="gz-sim-sensors-system">
+             <render_engine>ogre2</render_engine>
+        </plugin>
         <plugin name="gz::sim::systems::DiffDrive" filename="gz-sim-diff-drive-system">
             <left_joint>left_wheel_joint</left_joint>

Commit message: Before thrying to add realism

File: src/lawn_mower_bot/urdf/mower.urdf.xacro (robot description, xacro)
@@ -251,4 +251,33 @@
             <topic>/joint_states</topic>
         </plugin>
+        <plugin filename="gz-sim-particle-emitter-system" name="gz::sim::systems::ParticleEmitter">
+        </plugin>
+    </gazebo>
+    <!-- GRASS PARTICLE EMITTER (Simulates the blade cutting grass) -->
+    <link name="blade_link">
+        <pose>0 0 0.02 0 0 0</pose>
+    </link>
+    <joint name="blade_joint" type="fixed">
+        <parent link="base_link" />
+        <child link="blade_link" />
+        <origin xyz="-0.1 0 -0.05" rpy="0 0 0" />
+    </joint>
+    <gazebo reference="blade_link">
+        <particle_emitter name="grass_emitter" type="box">
+            <emitting>false</emitting>
+            <size>0.3 0.2 0</size>
+            <particle_size>0.02 0.02 0.02</particle_size>
+            <lifetime>2.0</lifetime>
+            <min_velocity>0.1</min_velocity>
+            <max_velocity>0.3</max_velocity>
+            <rate>200</rate>
+            <scale_rate>0</scale_rate>
+            <scatter_ratio>0.2</scatter_ratio>
+            <material>
+                <ambient>0.0 0.8 0.0 1.0</ambient>
+                <diffuse>0.0 0.8 0.0 1.0</diffuse>
+            </material>
+            <topic>/mower_blade_state</topic>
+        </particle_emitter>
     </gazebo>
 </robot>
